File: ThermorZigbeeController/hardware/kicad/thermor_zigbee_controller.kicad_sch (KiCad schematic)
At the start: 7 parts, among them U1 ESP32-C6-WROOM-1, U2 HT1621, U3 PC817, U4 HC-SR501

Commit message: Update
Parts:
- removed R2: 10k, Resistor_SMD:R_0603_1608Metric, symbol Device:R
- removed U4: HC-SR501, symbol PIR_Sensor
- C1: value 100nF -> 470uF; footprint Capacitor_SMD:C_0603_1608Metric -> Capacitor_THT:CP_Radial_D8.0mm_P3.50mm
- R1: value 1k -> 330; footprint Resistor_SMD:R_0603_1608Metric -> Resistor_SMD:R_0805_2012Metric
Connections:
- net GND: now also U1.20 (GND); no longer U1.19 (GND)
- no-connect marks 2 -> 0
Other:
- note removed: "Button Matrix"
- note removed: "ESP32-C6 ZIGBEE CONTROLLER FOR THERMOR EMOTION 4"
- note removed: "LCD Interface (HT1621)"
- note removed: "PIR Motion Sensor"
- note removed: "Power Supply"
- note removed: "Triac Control"
